Commit message: add limit property to wheel joints

File: urdf/navvis.xacro (robot description, xacro)
@@ -103,5 +103,5 @@
       <origin xyz=" -0.1 ${reflect * 0.4} 0.0" rpy=" ${-pi/2} 0.0 0.0" />
       <axis xyz="0 0 1" />
-      <!-- <limit effort="" velocity="" /> -->
+      <limit effort="${1E6}" velocity="${1E6}" />
     </joint>
   </xacro:macro>
@@ -125,4 +125,5 @@
     <origin xyz=" 0.1 0.0 0.0" rpy="${-pi/2} 0.0 0.0" />
     <axis xyz="0 0 1" />
+    <limit effort="${1E6}" velocity="${1E6}" />
   </joint>
   <xacro:include filename="$(find gazebo_plugins)/test/multi_robot_scenario/xacro/laser/hokuyo.xacro" />
